Commit message: import STL into URDF
Now the joint offset and link offset is tuned by hand. In the future, I
might use the CAD file to recalculate to be more precise.

File: spyndra_description/urdf/component.urdf (robot description, URDF)
Before this commit: robot component, 1 links, 0 joints
Links:
- link base_link: geometry collision mesh filename=package://learning_urdf/meshes/chassis.stl scale=0.001 0.001 0.001; visual mesh filename=package://learning_urdf/meshes/chassis.stl scale=0.001 0.001 0.001

File: spyndra_description/urdf/spyndra.urdf.xacro (robot description, xacro)
@@ -5,14 +5,31 @@
   <!-- stl offset -->
   <!-- component length -->
-  <xacro:property name="lc1" value="0.068"/>
-  <xacro:property name="lc2" value="0.0508"/>
+  <xacro:property name="lc1" value="0.061"/>
+  <xacro:property name="lc2" value="0.058"/>
   <xacro:property name="hc1" value="0.09441"/>
   <xacro:property name="hc2" value="0.01"/>
   <xacro:property name="lf" value="0.127"/>
   <xacro:property name="wf" value="0.0848"/>
-  <xacro:property name="hf" value="0.04"/>
+  <xacro:property name="hf" value="0.06"/>
   <xacro:property name="lt" value="0.18858"/>
   <xacro:property name="rt" value="0.017"/>
   <xacro:property name="dt" value="0.21227"/>
+  <!-- link offset -->
+  <xacro:property name="off_cx" value="-0.11" />
+  <xacro:property name="off_cy" value="-0.068" />
+  <xacro:property name="off_cz" value="0" />
+  <xacro:property name="off_fx" value="-0.00825" />
+  <xacro:property name="off_fy" value="0.0455" />
+  <xacro:property name="off_fz" value="-0.022" />
+  <xacro:property name="off_tx" value="0.1735" />
+  <xacro:property name="off_ty" value="0.0215" />
+  <xacro:property name="off_tz" value="-0.02" />
+  <!-- joint offset -->
+  <xacro:property name="jt_cx" value="0.0585" />
+  <xacro:property name="jt_cy" value="-0.003" />
+  <xacro:property name="jt_cz" value="0.047" />
+  <xacro:property name="jt_fx" value="0.111" />
+  <xacro:property name="jt_fy" value="0.003" />
+  <xacro:property name="jt_fz" value="0" />
   <!-- component mass -->
   <xacro:property name="mc" value="0.23069271"/>
@@ -35,5 +52,5 @@
         <mesh filename="package://spyndra_description/meshes/chassis.stl"     scale="0.001 0.001 0.001"/>
       </geometry>
-      <origin xyz="-0.11 -0.068 0" rpy="0 0 0"/>
+      <origin xyz="${off_cx} ${off_cy} ${off_cz}" rpy="0 0 0"/>
     </collision>
     <visual>
@@ -41,5 +58,5 @@
         <mesh filename="package://spyndra_description/meshes/chassis.stl"     scale="0.001 0.001 0.001"/>
       </geometry>
-      <origin xyz="-0.11 -0.068 0" rpy="0 0 0"/>
+      <origin xyz="${off_cx} ${off_cy} ${off_cz}" rpy="0 0 0"/>
       <material name="black"/>
     </visual>
@@ -55,15 +72,15 @@
     <collision>
       <geometry>
-        <mesh filename="package://spyndra_description/meshes/femur.stl"     scale="0.001 0.001 0.001"/>
-      </geometry>
-      <material name="red"/>
-      <origin xyz="-0.00825 0.0455 -0.022" rpy="3.1415926 -1.57075 0    "/>
-    </collision>
-    <visual>
-      <geometry>
-        <mesh filename="package://spyndra_description/meshes/femur.stl"     scale="0.001 0.001 0.001"/>
-      </geometry>
-      <material name="red"/>
-      <origin xyz="-0.00825 0.0455 -0.022" rpy="3.1415926 -1.57075 0    "/>
+        <mesh filename="package://spyndra_description/meshes/femur.stl" scale="0.001 0.001 0.001"/>
+      </geometry>
+      <material name="red"/>
+      <origin xyz="${off_fx} ${off_fy} ${off_fz}" rpy="${pi} ${-pi/2} 0"/>
+    </collision>
+    <visual>
+      <geometry>
+        <mesh filename="package://spyndra_description/meshes/femur.stl" scale="0.001 0.001 0.001"/>
+      </geometry>
+      <material name="red"/>
+      <origin xyz="${off_fx} ${off_fy} ${off_fz}" rpy="${pi} ${-pi/2} 0"/>
     </visual>
     <inertial>
@@ -81,15 +98,15 @@
     <collision>
       <geometry>
-        <mesh filename="package://spyndra_description/meshes/tibia.stl"     scale="0.001 0.001 0.001"/>
-      </geometry>
-      <material name="white"/>
-      <origin xyz="0.1735 0.0215 -0.02" rpy="1.57075 0 -1.57075"/>
-    </collision>
-    <visual>
-      <geometry>
-        <mesh filename="package://spyndra_description/meshes/tibia.stl"     scale="0.001 0.001 0.001"/>
-      </geometry>
-      <material name="white"/>
-      <origin xyz="0.1735 0.0215 -0.02" rpy="1.57075 0 -1.57075"/>
+        <mesh filename="package://spyndra_description/meshes/tibia.stl" scale="0.001 0.001 0.001"/>
+      </geometry>
+      <material name="white"/>
+      <origin xyz="${off_tx} ${off_ty} ${off_tz}" rpy="${pi/2} 0 ${-pi/2}"/>
+    </collision>
+    <visual>
+      <geometry>
+        <mesh filename="package://spyndra_description/meshes/tibia.stl" scale="0.001 0.001 0.001"/>
+      </geometry>
+      <material name="white"/>
+      <origin xyz="${off_tx} ${off_ty} ${off_tz}" rpy="${pi/2} 0 ${-pi/2}"/>
     </visual>
     <inertial>
@@ -107,24 +124,19 @@
     <collision>
       <geometry>
-        <box size="${lf} ${wf} ${hf}"/>
-      </geometry>
-      <material name="red"/>
-      <origin xyz="${lf/2} 0 0" rpy="0 0 0"/>
-    </collision>
-    <visual>
-      <geometry>
-        <box size="${lf} ${wf} ${hf}"/>
-      </geometry>
-      <material name="red"/>
-      <origin xyz="${lf/2} 0 0" rpy="0 0 0"/>
+        <mesh filename="package://spyndra_description/meshes/femur.stl" scale="0.001 0.001 0.001"/>
+      </geometry>
+      <material name="red"/>
+      <origin xyz="${off_fx} ${off_fy} ${off_fz}" rpy="${pi} ${-pi/2} 0"/>
+    </collision>
+    <visual>
+      <geometry>
+        <mesh filename="package://spyndra_description/meshes/femur.stl" scale="0.001 0.001 0.001"/>
+      </geometry>
+      <material name="red"/>
+      <origin xyz="${off_fx} ${off_fy} ${off_fz}" rpy="${pi} ${-pi/2} 0"/>
     </visual>
     <inertial>
       <origin xyz="0 0 ${hc1}"  rpy="0 0 0"/>
       <mass value="${mc}"/>
-      <!-- Simple geometry -->
-      <!--inertia ixx="${mc/12*(4*lc1*lc1+hc1*hc1)}" ixy="0"
-        iyy="${mc/12*(4*lc1*lc1+hc1*hc1)}" iyz="0"
-        izz="${mc/6*4*lc1*lc1}" ixz="0"/-->
-      <!-- From CAD file -->
       <inertia ixx="${0.00025261+mf*(fy*fy+fz*fz)}"
         ixy="${        0.0-mf*fx*fy}"
@@ -138,24 +150,19 @@
     <collision>
       <geometry>
-        <cylinder length="${lt}" radius="${rt}"/>
-      </geometry>
-      <material name="white"/>
-      <origin rpy="0 ${pi/2} 0" xyz="${lt/2} 0 0"/>
-    </collision>
-    <visual>
-      <geometry>
-        <cylinder length="${lt}" radius="${rt}"/>
-      </geometry>
-      <material name="white"/>
-      <origin rpy="0 ${pi/2} 0" xyz="${lt/2} 0 0"/>
+        <mesh filename="package://spyndra_description/meshes/tibia.stl" scale="0.001 0.001 0.001"/>
+      </geometry>
+      <material name="white"/>
+      <origin xyz="${off_tx} ${off_ty} ${off_tz}" rpy="${pi/2} 0 ${-pi/2}"/>
+    </collision>
+    <visual>
+      <geometry>
+        <mesh filename="package://spyndra_description/meshes/tibia.stl" scale="0.001 0.001 0.001"/>
+      </geometry>
+      <material name="white"/>
+      <origin xyz="${off_tx} ${off_ty} ${off_tz}" rpy="${pi/2} 0 ${-pi/2}"/>
     </visual>
     <inertial>
       <origin xyz="${lt/2} 0 0" rpy="0 0 0"/>
       <mass value="${mt}"/>
-      <!-- Simple geometry -->
-      <!--inertia ixx="${mt/2*rt*rt}" ixy="0"
-        iyy="${mt/3*lt*lt}" iyz="0"
-        izz="${mt/3*lt*lt}" ixz="0"/-->
-      <!-- From CAD file -->
       <inertia ixx="${0.00021435+mt*(ty*ty+tz*tz)}"
         ixy="${-0.00000128-mt*tx*ty}"
@@ -169,24 +176,19 @@
     <collision>
       <geometry>
-        <box size="${lf} ${wf} ${hf}"/>
-      </geometry>
-      <material name="red"/>
-      <origin xyz="${lf/2} 0 0" rpy="0 0 0"/>
-    </collision>
-    <visual>
-      <geometry>
-        <box size="${lf} ${wf} ${hf}"/>
-      </geometry>
-      <material name="red"/>
-      <origin xyz="${lf/2} 0 0" rpy="0 0 0"/>
+        <mesh filename="package://spyndra_description/meshes/femur.stl" scale="0.001 0.001 0.001"/>
+      </geometry>
+      <material name="red"/>
+      <origin xyz="${off_fx} ${off_fy} ${off_fz}" rpy="${pi} ${-pi/2} 0"/>
+    </collision>
+    <visual>
+      <geometry>
+        <mesh filename="package://spyndra_description/meshes/femur.stl" scale="0.001 0.001 0.001"/>
+      </geometry>
+      <material name="red"/>
+      <origin xyz="${off_fx} ${off_fy} ${off_fz}" rpy="${pi} ${-pi/2} 0"/>
     </visual>
     <inertial>
       <origin xyz="0 0 ${hc1}"  rpy="0 0 0"/>
       <mass value="${mc}"/>
-      <!-- Simple geometry -->
-      <!--inertia ixx="${mc/12*(4*lc1*lc1+hc1*hc1)}" ixy="0"
-        iyy="${mc/12*(4*lc1*lc1+hc1*hc1)}" iyz="0"
-        izz="${mc/6*4*lc1*lc1}" ixz="0"/-->
-      <!-- From CAD file -->
       <inertia ixx="${0.00025261+mf*(fy*fy+fz*fz)}"
         ixy="${        0.0-mf*fx*fy}"
@@ -207,24 +209,19 @@
     <collision>
       <geometry>
-        <cylinder length="${lt}" radius="${rt}"/>
-      </geometry>
-      <material name="white"/>
-      <origin rpy="0 ${pi/2} 0" xyz="${lt/2} 0 0"/>
-    </collision>
-    <visual>
-      <geometry>
-        <cylinder length="${lt}" radius="${rt}"/>
-      </geometry>
-      <material name="white"/>
-      <origin rpy="0 ${pi/2} 0" xyz="${lt/2} 0 0"/>
+        <mesh filename="package://spyndra_description/meshes/tibia.stl" scale="0.001 0.001 0.001"/>
+      </geometry>
+      <material name="white"/>
+      <origin xyz="${off_tx} ${off_ty} ${off_tz}" rpy="${pi/2} 0 ${-pi/2}"/>
+    </collision>
+    <visual>
+      <geometry>
+        <mesh filename="package://spyndra_description/meshes/tibia.stl" scale="0.001 0.001 0.001"/>
+      </geometry>
+      <material name="white"/>
+      <origin xyz="${off_tx} ${off_ty} ${off_tz}" rpy="${pi/2} 0 ${-pi/2}"/>
     </visual>
     <inertial>
       <origin xyz="${lt/2} 0 0" rpy="0 0 0"/>
       <mass value="${mt}"/>
-      <!-- Simple geometry -->
-      <!--inertia ixx="${mt/2*rt*rt}" ixy="0"
-        iyy="${mt/3*lt*lt}" iyz="0"
-        izz="${mt/3*lt*lt}" ixz="0"/-->
-      <!-- From CAD file -->
       <inertia ixx="${0.00021435+mt*(ty*ty+tz*tz)}"
         ixy="${-0.00000128-mt*tx*ty}"
@@ -238,24 +235,19 @@
     <collision>
       <geometry>
-        <box size="${lf} ${wf} ${hf}"/>
-      </geometry>
-      <material name="red"/>
-      <origin xyz="${lf/2} 0 0" rpy="0 0 0"/>
-    </collision>
-    <visual>
-      <geometry>
-        <box size="${lf} ${wf} ${hf}"/>
-      </geometry>
-      <material name="red"/>
-      <origin xyz="${lf/2} 0 0" rpy="0 0 0"/>
+        <mesh filename="package://spyndra_description/meshes/femur.stl" scale="0.001 0.001 0.001"/>
+      </geometry>
+      <material name="red"/>
+      <origin xyz="${off_fx} ${off_fy} ${off_fz}" rpy="${pi} ${-pi/2} 0"/>
+    </collision>
+    <visual>
+      <geometry>
+        <mesh filename="package://spyndra_description/meshes/femur.stl" scale="0.001 0.001 0.001"/>
+      </geometry>
+      <material name="red"/>
+      <origin xyz="${off_fx} ${off_fy} ${off_fz}" rpy="${pi} ${-pi/2} 0"/>
     </visual>
     <inertial>
       <origin xyz="0 0 ${hc1}"  rpy="0 0 0"/>
       <mass value="${mc}"/>
-      <!-- Simple geometry -->
-      <!--inertia ixx="${mc/12*(4*lc1*lc1+hc1*hc1)}" ixy="0"
-        iyy="${mc/12*(4*lc1*lc1+hc1*hc1)}" iyz="0"
-        izz="${mc/6*4*lc1*lc1}" ixz="0"/-->
-      <!-- From CAD file -->
       <inertia ixx="${0.00025261+mf*(fy*fy+fz*fz)}"
         ixy="${        0.0-mf*fx*fy}"
@@ -269,24 +261,19 @@
     <collision>
       <geometry>
-        <cylinder length="${lt}" radius="${rt}"/>
-      </geometry>
-      <material name="white"/>
-      <origin rpy="0 ${pi/2} 0" xyz="${lt/2} 0 0"/>
-    </collision>
-    <visual>
-      <geometry>
-        <cylinder length="${lt}" radius="${rt}"/>
-      </geometry>
-      <material name="white"/>
-      <origin rpy="0 ${pi/2} 0" xyz="${lt/2} 0 0"/>
+        <mesh filename="package://spyndra_description/meshes/tibia.stl" scale="0.001 0.001 0.001"/>
+      </geometry>
+      <material name="white"/>
+      <origin xyz="${off_tx} ${off_ty} ${off_tz}" rpy="${pi/2} 0 ${-pi/2}"/>
+    </collision>
+    <visual>
+      <geometry>
+        <mesh filename="package://spyndra_description/meshes/tibia.stl" scale="0.001 0.001 0.001"/>
+      </geometry>
+      <material name="white"/>
+      <origin xyz="${off_tx} ${off_ty} ${off_tz}" rpy="${pi/2} 0 ${-pi/2}"/>
     </visual>
     <inertial>
       <origin xyz="${lt/2} 0 0" rpy="0 0 0"/>
       <mass value="${mt}"/>
-      <!-- Simple geometry -->
-      <!--inertia ixx="${mt/2*rt*rt}" ixy="0"
-        iyy="${mt/3*lt*lt}" iyz="0"
-        izz="${mt/3*lt*lt}" ixz="0"/-->
-      <!-- From CAD file -->
       <inertia ixx="${0.00021435+mt*(ty*ty+tz*tz)}"
         ixy="${-0.00000128-mt*tx*ty}"
@@ -301,5 +288,5 @@
     <child link="femur_1"/>
     <axis xyz="0 1 0"/>
-    <origin rpy="0 0 0" xyz="${lc2} 0 ${hc2+hc1/2}"/>
+    <origin rpy="0 0 0" xyz="${jt_cx} ${jt_cy} ${jt_cz}"/>
     <limit effort="1000.0" lower="-0.5" upper="0.8" velocity="0.5"/>
   </joint>
@@ -308,5 +295,5 @@
     <child link="tibia_1"/>
     <axis xyz="0 1 0"/>
-    <origin rpy="0 ${dt} 0" xyz="${lf} 0 0"/>
+    <origin rpy="0 0 0" xyz="${jt_fx} ${jt_fy} ${jt_fz}"/>
     <limit effort="1000.0" lower="-0.5" upper="0.8" velocity="0.5"/>
   </joint>
@@ -315,5 +302,5 @@
     <child link="femur_2"/>
     <axis xyz="0 1 0"/>
-    <origin rpy="0 0 ${-pi/2}" xyz="0 ${-lc2} ${hc2+hc1/2}"/>
+    <origin rpy="0 0 ${-pi/2}" xyz="${jt_cy} ${-jt_cx} ${jt_cz}"/>
     <limit effort="1000.0" lower="-0.5" upper="0.8" velocity="0.5"/>
   </joint>
@@ -322,5 +309,5 @@
     <child link="tibia_2"/>
     <axis xyz="0 1 0"/>
-    <origin rpy="0 ${dt} 0" xyz="${lf} 0 0"/>
+    <origin rpy="0 0 0" xyz="${jt_fx} ${jt_fy} ${jt_fz}"/>
     <limit effort="1000.0" lower="-0.5" upper="0.8" velocity="0.5"/>
   </joint>
@@ -329,5 +316,5 @@
     <child link="femur_3"/>
     <axis xyz="0 1 0"/>
-    <origin rpy="0 0 ${-pi}" xyz="${-lc2} 0 ${hc2+hc1/2}"/>
+    <origin rpy="0 0 ${-pi}" xyz="${-jt_cx} ${-jt_cy} ${jt_cz}"/>
     <limit effort="1000.0" lower="-0.5" upper="0.8" velocity="0.5"/>
   </joint>
@@ -336,5 +323,5 @@
     <child link="tibia_3"/>
     <axis xyz="0 1 0"/>
-    <origin rpy="0 ${dt} 0" xyz="${lf} 0 0"/>
+    <origin rpy="0 0 0" xyz="${jt_fx} ${jt_fy} ${jt_fz}"/>
     <limit effort="1000.0" lower="-0.5" upper="0.8" velocity="0.5"/>
   </joint>
@@ -343,5 +330,5 @@
     <child link="femur_4"/>
     <axis xyz="0 1 0"/>
-    <origin rpy="0 0 ${pi/2}" xyz="0 ${lc2} ${hc2+hc1/2}"/>
+    <origin rpy="0 0 ${pi/2}" xyz="${-jt_cy} ${jt_cx} ${jt_cz}"/>
     <limit effort="1000.0" lower="-0.5" upper="0.8" velocity="0.5"/>
   </joint>
@@ -350,5 +337,5 @@
     <child link="tibia_4"/>
     <axis xyz="0 1 0"/>
-    <origin rpy="0 ${dt} 0" xyz="${lf} 0 0"/>
+    <origin rpy="0 0 0" xyz="${jt_fx} ${jt_fy} ${jt_fz}"/>
     <limit effort="1000.0" lower="-0.5" upper="0.8" velocity="0.5"/>
   </joint>
