Commit message: feat: motor controller for femur1 and tibia1
Ref: http://gazebosim.org/tutorials/?tut=ros_control
Add position controller to femur1 and tibia1. If this works out,
one can use rqt's gui to send motor command.

Task to follow up:
 - Tune PID paramters
 - Add position controller to other joints

File: spyndra_description/urdf/spyndra.urdf.xacro (robot description, xacro)
@@ -1,6 +1,6 @@
 <?xml version="1.0"?>
-<robot name="simple_model" xmlns:xacro="http://www.ros.org/wiki/xacro">
-  <!-- color -->
-  <material name="blue">
+<robot name="spyndra" xmlns:xacro="http://www.ros.org/wiki/xacro">
+  <!-- Rviz colors -->
+  <!--material name="blue">
     <color rgba="0 0 0.8 1"/>
   </material>
@@ -13,5 +13,5 @@
   <material name="white">
     <color rgba="1 1 1 1"/>
-  </material>
+  </material-->
   <!-- constants -->
   <xacro:property name="lc1" value="0.068"/>
@@ -29,4 +29,7 @@
   <xacro:property name="mf" value="0.16076767"/>
   <xacro:property name="mt" value="0.08869082"/>
+  <!-- Import all Gazebo-customization elements -->
+  <xacro:include filename="$(find spyndra_description)/urdf/spyndra.gazebo" />
+  <xacro:include filename="$(find spyndra_description)/urdf/materials.xacro" />
   <!-- links -->
   <link name="base_link">
@@ -35,5 +38,5 @@
         <box size="${2*lc1} ${2*lc1} ${hc1}" />
       </geometry>
-      <origin rpy="0 0 0" xyz="0 0 ${hc2}"/>
+      <origin rpy="0 0 0" xyz="0 0 ${hc1/2}"/>
     </collision>
     <visual>
@@ -299,13 +302,25 @@
     <limit effort="1000.0" lower="-0.5" upper="0.8" velocity="0.5"/>
   </joint>
-  <gazebo>
-    <plugin name="imu_plugin" filename="libgazebo_ros_imu.so">
-      <alwaysOn>true</alwaysOn>
-      <bodyName>base_link</bodyName>
-      <topicName>imu</topicName>
-      <serviceName>imu_service</serviceName>
-      <gaussianNoise>0.0</gaussianNoise>
-      <updateRate>20.0</updateRate>
-    </plugin>
-  </gazebo>
+  <!-- Actuators -->
+  <transmission name="tran_f1">
+    <type>transmission_interface/SimpleTransmission</type>
+    <joint name="motor_f1">
+      <!--hardwareInterface>EffortJointInterface</hardwareInterface-->
+      <hardwareInterface>EffortJointInterface</hardwareInterface>
+    </joint>
+    <actuator name="servo_f1">
+      <hardwareInterface>EffortJointInterface</hardwareInterface>
+      <mechanicalReduction>1</mechanicalReduction>
+    </actuator>
+  </transmission>
+  <transmission name="tran_t1">
+    <type>transmission_interface/SimpleTransmission</type>
+    <joint name="motor_t1">
+      <hardwareInterface>EffortJointInterface</hardwareInterface>
+    </joint>
+    <actuator name="servo_t1">
+      <hardwareInterface>EffortJointInterface</hardwareInterface>
+      <mechanicalReduction>1</mechanicalReduction>
+    </actuator>
+  </transmission>
 </robot>

Commit message: feat: add motor to leg2-4
Add motor to femur2-4, tibia2-4
Now we can use rqt_gui to send motor command.
Suggested locomotion are:

60Hz - sin(i/60)+150  for femurs
60Hz - sin(i/60)+50   for tibias

Follow ups:
 - Write command publisher

File: spyndra_description/urdf/spyndra.urdf.xacro (robot description, xacro)
@@ -324,3 +324,63 @@
     </actuator>
   </transmission>
+  <transmission name="tran_f2">
+    <type>transmission_interface/SimpleTransmission</type>
+    <joint name="motor_f2">
+      <hardwareInterface>EffortJointInterface</hardwareInterface>
+    </joint>
+    <actuator name="servo_f2">
+      <hardwareInterface>EffortJointInterface</hardwareInterface>
+      <mechanicalReduction>1</mechanicalReduction>
+    </actuator>
+  </transmission>
+  <transmission name="tran_t2">
+    <type>transmission_interface/SimpleTransmission</type>
+    <joint name="motor_t2">
+      <hardwareInterface>EffortJointInterface</hardwareInterface>
+    </joint>
+    <actuator name="servo_t2">
+      <hardwareInterface>EffortJointInterface</hardwareInterface>
+      <mechanicalReduction>1</mechanicalReduction>
+    </actuator>
+  </transmission>
+  <transmission name="tran_f3">
+    <type>transmission_interface/SimpleTransmission</type>
+    <joint name="motor_f3">
+      <hardwareInterface>EffortJointInterface</hardwareInterface>
+    </joint>
+    <actuator name="servo_f3">
+      <hardwareInterface>EffortJointInterface</hardwareInterface>
+      <mechanicalReduction>1</mechanicalReduction>
+    </actuator>
+  </transmission>
+  <transmission name="tran_t3">
+    <type>transmission_interface/SimpleTransmission</type>
+    <joint name="motor_t3">
+      <hardwareInterface>EffortJointInterface</hardwareInterface>
+    </joint>
+    <actuator name="servo_t3">
+      <hardwareInterface>EffortJointInterface</hardwareInterface>
+      <mechanicalReduction>1</mechanicalReduction>
+    </actuator>
+  </transmission>
+  <transmission name="tran_f4">
+    <type>transmission_interface/SimpleTransmission</type>
+    <joint name="motor_f4">
+      <hardwareInterface>EffortJointInterface</hardwareInterface>
+    </joint>
+    <actuator name="servo_f4">
+      <hardwareInterface>EffortJointInterface</hardwareInterface>
+      <mechanicalReduction>1</mechanicalReduction>
+    </actuator>
+  </transmission>
+  <transmission name="tran_t4">
+    <type>transmission_interface/SimpleTransmission</type>
+    <joint name="motor_t4">
+      <hardwareInterface>EffortJointInterface</hardwareInterface>
+    </joint>
+    <actuator name="servo_t4">
+      <hardwareInterface>EffortJointInterface</hardwareInterface>
+      <mechanicalReduction>1</mechanicalReduction>
+    </actuator>
+  </transmission>
 </robot>

Commit message: feat: visualize robot description file
Before calculating detailed inertia, I moved the tool from learning_urdf
package to here. The new launch file should be able to display the robot
in RViz.

Following works include calibrating joint angle limits and calculating
moment of inertia.

File: spyndra_description/urdf/spyndra.urdf.xacro (robot description, xacro)
@@ -1,17 +1,4 @@
 <?xml version="1.0"?>
 <robot name="spyndra" xmlns:xacro="http://www.ros.org/wiki/xacro">
-  <!-- Rviz colors -->
-  <!--material name="blue">
-    <color rgba="0 0 0.8 1"/>
-  </material>
-  <material name="black">
-    <color rgba="0 0 0 1"/>
-  </material>
-  <material name="red">
-    <color rgba="1 0 0 1"/>
-  </material>
-  <material name="white">
-    <color rgba="1 1 1 1"/>
-  </material-->
   <!-- constants -->
   <xacro:property name="lc1" value="0.068"/>
@@ -26,7 +13,7 @@
   <xacro:property name="dt" value="0.21227"/>
   <xacro:property name="pi" value="3.1415926535897931"/>
-  <xacro:property name="mc" value="0.18225809"/>
-  <xacro:property name="mf" value="0.16076767"/>
-  <xacro:property name="mt" value="0.08869082"/>
+  <xacro:property name="mc" value="0.23069271"/>
+  <xacro:property name="mf" value="0.20096365"/>
+  <xacro:property name="mt" value="0.10764861"/>
   <!-- Import all Gazebo-customization elements -->
   <xacro:include filename="$(find spyndra_description)/urdf/spyndra.gazebo" />

Commit message: feat: calibrate inertia from CAD file
Previously I used simple geometry assumption to calculate moment of
inertia. However, this assumption might lead to very different IMU
measurement. Hence, I calculated to inertia about center of mass by
Solidworks and apply offset calculate to account for non-central
rotation.

Followup: verify the IMU measurement is closer to the real robot.

File: spyndra_description/urdf/spyndra.urdf.xacro (robot description, xacro)
@@ -2,4 +2,6 @@
 <robot name="spyndra" xmlns:xacro="http://www.ros.org/wiki/xacro">
   <!-- constants -->
+  <xacro:property name="pi" value="3.1415926535897931"/>
+  <!-- component length -->
   <xacro:property name="lc1" value="0.068"/>
   <xacro:property name="lc2" value="0.0508"/>
@@ -12,8 +14,15 @@
   <xacro:property name="rt" value="0.017"/>
   <xacro:property name="dt" value="0.21227"/>
-  <xacro:property name="pi" value="3.1415926535897931"/>
+  <!-- component mass -->
   <xacro:property name="mc" value="0.23069271"/>
   <xacro:property name="mf" value="0.20096365"/>
   <xacro:property name="mt" value="0.10764861"/>
+  <!-- inertia offsets -->
+  <xacro:property name="fx" value="-0.0006" />
+  <xacro:property name="fy" value="0.0" />
+  <xacro:property name="fz" value="-0.05762" />
+  <xacro:property name="tx" value="-0.06001" />
+  <xacro:property name="ty" value="0.0" />
+  <xacro:property name="tz" value="0.0102" />
   <!-- Import all Gazebo-customization elements -->
   <xacro:include filename="$(find spyndra_description)/urdf/spyndra.gazebo" />
@@ -37,7 +46,12 @@
       <origin xyz="0 0 ${hc1}"  rpy="0 0 0"/>
       <mass value="${mc}"/>
-      <inertia ixx="${mc/12*(4*lc1*lc1+hc1*hc1)}" ixy="0"
+      <!-- Simple geometry -->
+      <!--inertia ixx="${mc/12*(4*lc1*lc1+hc1*hc1)}" ixy="0"
         iyy="${mc/12*(4*lc1*lc1+hc1*hc1)}" iyz="0"
-        izz="${mc/6*4*lc1*lc1}" ixz="0"/>
+        izz="${mc/6*4*lc1*lc1}" ixz="0"/-->
+      <!-- From CAD file -->
+      <inertia ixx="0.00029636" ixy="0.00000019"
+        iyy="0.00028197" iyz = "-0.00000269"
+        izz="0.00044786" ixz="-0.00000106" />
     </inertial>
   </link>
@@ -60,7 +74,15 @@
       <origin xyz="${lf/2} 0 0" rpy="0 0 0"/>
       <mass value="${mf}"/>
-      <inertia ixx="${mf/12*(wf*wf+hf*hf)}" ixy="0"
+      <!-- Simple geometry -->
+      <!--inertia ixx="${mf/12*(wf*wf+hf*hf)}" ixy="0"
         iyy="${mf/3*lf*lf+mf/12*wf*wf}" iyz="0"
-        izz="${mf/3*lf*lf+mf/12*hf*hf}" ixz="0"/>
+        izz="${mf/3*lf*lf+mf/12*hf*hf}" ixz="0"/-->
+      <!-- From CAD file -->
+      <inertia ixx="${0.00025261+mf*(fy*fy+fz*fz)}"
+        ixy="${        0.0-mf*fx*fy}"
+        iyy="${ 0.00014944+mf*(fx*fx+fz*fz)}"
+        iyz="${-0.00000002-mf*fy*fz}"
+        izz="${ 0.00013756+mf*(fx*fx+fy*fy)}"
+        ixz="${-0.00000601-mf*fx*fz}" />
     </inertial>
   </link>
@@ -80,4 +102,112 @@
       <origin rpy="0 ${pi/2} 0" xyz="${lt/2} 0 0"/>
     </visual>
+    <inertial>
+      <origin xyz="${lt/2} 0 0" rpy="0 0 0"/>
+      <mass value="${mt}"/>
+      <!-- Simple geometry -->
+      <!--inertia ixx="${mt/2*rt*rt}" ixy="0"
+        iyy="${mt/3*lt*lt}" iyz="0"
+        izz="${mt/3*lt*lt}" ixz="0"/ -->
+      <!-- From CAD file -->
+      <inertia ixx="${0.00021435+mt*(ty*ty+tz*tz)}"
+        ixy="${-0.00000128-mt*tx*ty}"
+        iyy="${ 0.00019560+mt*(tx*tx+tz*tz)}"
+        iyz="${-0.00005856-mt*ty*tz}"
+        izz="${ 0.00004159+mt*(tx*tx+ty*ty)}"
+        ixz="${ 0.00000606-mt*tx*tz}" />
+    </inertial>
+  </link>
+  <link name="femur_2">
+    <collision>
+      <geometry>
+        <box size="${lf} ${wf} ${hf}"/>
+      </geometry>
+      <material name="red"/>
+      <origin xyz="${lf/2} 0 0" rpy="0 0 0"/>
+    </collision>
+    <visual>
+      <geometry>
+        <box size="${lf} ${wf} ${hf}"/>
+      </geometry>
+      <material name="red"/>
+      <origin xyz="${lf/2} 0 0" rpy="0 0 0"/>
+    </visual>
+    <inertial>
+      <origin xyz="0 0 ${hc1}"  rpy="0 0 0"/>
+      <mass value="${mc}"/>
+      <!-- Simple geometry -->
+      <!--inertia ixx="${mc/12*(4*lc1*lc1+hc1*hc1)}" ixy="0"
+        iyy="${mc/12*(4*lc1*lc1+hc1*hc1)}" iyz="0"
+        izz="${mc/6*4*lc1*lc1}" ixz="0"/-->
+      <!-- From CAD file -->
+      <inertia ixx="${0.00025261+mf*(fy*fy+fz*fz)}"
+        ixy="${        0.0-mf*fx*fy}"
+        iyy="${ 0.00014944+mf*(fx*fx+fz*fz)}"
+        iyz="${-0.00000002-mf*fy*fz}"
+        izz="${ 0.00013756+mf*(fx*fx+fy*fy)}"
+        ixz="${-0.00000601-mf*fx*fz}" />
+    </inertial>
+  </link>
+  <link name="tibia_2">
+    <collision>
+      <geometry>
+        <cylinder length="${lt}" radius="${rt}"/>
+      </geometry>
+      <material name="white"/>
+      <origin rpy="0 ${pi/2} 0" xyz="${lt/2} 0 0"/>
+    </collision>
+    <visual>
+      <geometry>
+        <cylinder length="${lt}" radius="${rt}"/>
+      </geometry>
+      <material name="white"/>
+      <origin rpy="0 ${pi/2} 0" xyz="${lt/2} 0 0"/>
+    </visual>
+    <inertial>
+      <origin xyz="${lt/2} 0 0" rpy="0 0 0"/>
+      <mass value="${mt}"/>
+      <!-- Simple geometry -->
+      <!--inertia ixx="${mt/2*rt*rt}" ixy="0"
+        iyy="${mt/3*lt*lt}" iyz="0"
+        izz="${mt/3*lt*lt}" ixz="0"/-->
+      <!-- From CAD file -->
+      <inertia ixx="${0.00021435+mt*(ty*ty+tz*tz)}"
+        ixy="${-0.00000128-mt*tx*ty}"
+        iyy="${ 0.00019560+mt*(tx*tx+tz*tz)}"
+        iyz="${-0.00005856-mt*ty*tz}"
+        izz="${ 0.00004159+mt*(tx*tx+ty*ty)}"
+        ixz="${ 0.00000606-mt*tx*tz}" />
+    </inertial>
+  </link>
+  <link name="femur_3">
+    <collision>
+      <geometry>
+        <box size="${lf} ${wf} ${hf}"/>
+      </geometry>
+      <material name="red"/>
+      <origin xyz="${lf/2} 0 0" rpy="0 0 0"/>
+    </collision>
+    <visual>
+      <geometry>
+        <box size="${lf} ${wf} ${hf}"/>
+      </geometry>
+      <material name="red"/>
+      <origin xyz="${lf/2} 0 0" rpy="0 0 0"/>
+    </visual>
+    <inertial>
+      <origin xyz="0 0 ${hc1}"  rpy="0 0 0"/>
+      <mass value="${mc}"/>
+      <!-- Simple geometry -->
+      <!--inertia ixx="${mc/12*(4*lc1*lc1+hc1*hc1)}" ixy="0"
+        iyy="${mc/12*(4*lc1*lc1+hc1*hc1)}" iyz="0"
+        izz="${mc/6*4*lc1*lc1}" ixz="0"/-->
+      <!-- From CAD file -->
+      <inertia ixx="${0.00025261+mf*(fy*fy+fz*fz)}"
+        ixy="${        0.0-mf*fx*fy}"
+        iyy="${ 0.00014944+mf*(fx*fx+fz*fz)}"
+        iyz="${-0.00000002-mf*fy*fz}"
+        izz="${ 0.00013756+mf*(fx*fx+fy*fy)}"
+        ixz="${-0.00000601-mf*fx*fz}" />
+    </inertial>
     <inertial>
       <origin xyz="${lt/2} 0 0" rpy="0 0 0"/>
@@ -88,5 +218,36 @@
     </inertial>
   </link>
-  <link name="femur_2">
+  <link name="tibia_3">
+    <collision>
+      <geometry>
+        <cylinder length="${lt}" radius="${rt}"/>
+      </geometry>
+      <material name="white"/>
+      <origin rpy="0 ${pi/2} 0" xyz="${lt/2} 0 0"/>
+    </collision>
+    <visual>
+      <geometry>
+        <cylinder length="${lt}" radius="${rt}"/>
+      </geometry>
+      <material name="white"/>
+      <origin rpy="0 ${pi/2} 0" xyz="${lt/2} 0 0"/>
+    </visual>
+    <inertial>
+      <origin xyz="${lt/2} 0 0" rpy="0 0 0"/>
+      <mass value="${mt}"/>
+      <!-- Simple geometry -->
+      <!--inertia ixx="${mt/2*rt*rt}" ixy="0"
+        iyy="${mt/3*lt*lt}" iyz="0"
+        izz="${mt/3*lt*lt}" ixz="0"/-->
+      <!-- From CAD file -->
+      <inertia ixx="${0.00021435+mt*(ty*ty+tz*tz)}"
+        ixy="${-0.00000128-mt*tx*ty}"
+        iyy="${ 0.00019560+mt*(tx*tx+tz*tz)}"
+        iyz="${-0.00005856-mt*ty*tz}"
+        izz="${ 0.00004159+mt*(tx*tx+ty*ty)}"
+        ixz="${ 0.00000606-mt*tx*tz}" />
+    </inertial>
+  </link>
+  <link name="femur_4">
     <collision>
       <geometry>
@@ -106,10 +267,18 @@
       <origin xyz="0 0 ${hc1}"  rpy="0 0 0"/>
       <mass value="${mc}"/>
-      <inertia ixx="${mc/12*(4*lc1*lc1+hc1*hc1)}" ixy="0"
+      <!-- Simple geometry -->
+      <!--inertia ixx="${mc/12*(4*lc1*lc1+hc1*hc1)}" ixy="0"
         iyy="${mc/12*(4*lc1*lc1+hc1*hc1)}" iyz="0"
-        izz="${mc/6*4*lc1*lc1}" ixz="0"/>
-    </inertial>
-  </link>
-  <link name="tibia_2">
+        izz="${mc/6*4*lc1*lc1}" ixz="0"/-->
+      <!-- From CAD file -->
+      <inertia ixx="${0.00025261+mf*(fy*fy+fz*fz)}"
+        ixy="${        0.0-mf*fx*fy}"
+        iyy="${ 0.00014944+mf*(fx*fx+fz*fz)}"
+        iyz="${-0.00000002-mf*fy*fz}"
+        izz="${ 0.00013756+mf*(fx*fx+fy*fy)}"
+        ixz="${-0.00000601-mf*fx*fz}" />
+    </inertial>
+  </link>
+  <link name="tibia_4">
     <collision>
       <geometry>
@@ -129,106 +298,15 @@
       <origin xyz="${lt/2} 0 0" rpy="0 0 0"/>
       <mass value="${mt}"/>
-      <inertia ixx="${mt/2*rt*rt}" ixy="0"
+      <!-- Simple geometry -->
+      <!--inertia ixx="${mt/2*rt*rt}" ixy="0"
         iyy="${mt/3*lt*lt}" iyz="0"
-        izz="${mt/3*lt*lt}" ixz="0"/>
-    </inertial>
-  </link>
-  <link name="femur_3">
-    <collision>
-      <geometry>
-        <box size="${lf} ${wf} ${hf}"/>
-      </geometry>
-      <material name="red"/>
-      <origin xyz="${lf/2} 0 0" rpy="0 0 0"/>
-    </collision>
-    <visual>
-      <geometry>
-        <box size="${lf} ${wf} ${hf}"/>
-      </geometry>
-      <material name="red"/>
-      <origin xyz="${lf/2} 0 0" rpy="0 0 0"/>
-    </visual>
-    <inertial>
-      <origin xyz="0 0 ${hc1}"  rpy="0 0 0"/>
-      <mass value="${mc}"/>
-      <inertia ixx="${mc/12*(4*lc1*lc1+hc1*hc1)}" ixy="0"
-        iyy="${mc/12*(4*lc1*lc1+hc1*hc1)}" iyz="0"
-        izz="${mc/6*4*lc1*lc1}" ixz="0"/>
-    </inertial>
-    <inertial>
-      <origin xyz="${lt/2} 0 0" rpy="0 0 0"/>
-      <mass value="${mt}"/>
-      <inertia ixx="${mt/2*rt*rt}" ixy="0"
-        iyy="${mt/3*lt*lt}" iyz="0"
-        izz="${mt/3*lt*lt}" ixz="0"/>
-    </inertial>
-  </link>
-  <link name="tibia_3">
-    <collision>
-      <geometry>
-        <cylinder length="${lt}" radius="${rt}"/>
-      </geometry>
-      <material name="white"/>
-      <origin rpy="0 ${pi/2} 0" xyz="${lt/2} 0 0"/>
-    </collision>
-    <visual>
-      <geometry>
-        <cylinder length="${lt}" radius="${rt}"/>
-      </geometry>
-      <material name="white"/>
-      <origin rpy="0 ${pi/2} 0" xyz="${lt/2} 0 0"/>
-    </visual>
-    <inertial>
-      <origin xyz="${lt/2} 0 0" rpy="0 0 0"/>
-      <mass value="${mt}"/>
-      <inertia ixx="${mt/2*rt*rt}" ixy="0"
-        iyy="${mt/3*lt*lt}" iyz="0"
-        izz="${mt/3*lt*lt}" ixz="0"/>
-    </inertial>
-  </link>
-  <link name="femur_4">
-    <collision>
-      <geometry>
-        <box size="${lf} ${wf} ${hf}"/>
-      </geometry>
-      <material name="red"/>
-      <origin xyz="${lf/2} 0 0" rpy="0 0 0"/>
-    </collision>
-    <visual>
-      <geometry>
-        <box size="${lf} ${wf} ${hf}"/>
-      </geometry>
-      <material name="red"/>
-      <origin xyz="${lf/2} 0 0" rpy="0 0 0"/>
-    </visual>
-    <inertial>
-      <origin xyz="0 0 ${hc1}"  rpy="0 0 0"/>
-      <mass value="${mc}"/>
-      <inertia ixx="${mc/12*(4*lc1*lc1+hc1*hc1)}" ixy="0"
-        iyy="${mc/12*(4*lc1*lc1+hc1*hc1)}" iyz="0"
-        izz="${mc/6*4*lc1*lc1}" ixz="0"/>
-    </inertial>
-  </link>
-  <link name="tibia_4">
-    <collision>
-      <geometry>
-        <cylinder length="${lt}" radius="${rt}"/>
-      </geometry>
-      <material name="white"/>
-      <origin rpy="0 ${pi/2} 0" xyz="${lt/2} 0 0"/>
-    </collision>
-    <visual>
-      <geometry>
-        <cylinder length="${lt}" radius="${rt}"/>
-      </geometry>
-      <material name="white"/>
-      <origin rpy="0 ${pi/2} 0" xyz="${lt/2} 0 0"/>
-    </visual>
-    <inertial>
-      <origin xyz="${lt/2} 0 0" rpy="0 0 0"/>
-      <mass value="${mt}"/>
-      <inertia ixx="${mt/2*rt*rt}" ixy="0"
-        iyy="${mt/3*lt*lt}" iyz="0"
-        izz="${mt/3*lt*lt}" ixz="0"/>
+        izz="${mt/3*lt*lt}" ixz="0"/-->
+      <!-- From CAD file -->
+      <inertia ixx="${0.00021435+mt*(ty*ty+tz*tz)}"
+        ixy="${-0.00000128-mt*tx*ty}"
+        iyy="${ 0.00019560+mt*(tx*tx+tz*tz)}"
+        iyz="${-0.00005856-mt*ty*tz}"
+        izz="${ 0.00004159+mt*(tx*tx+ty*ty)}"
+        ixz="${ 0.00000606-mt*tx*tz}" />
     </inertial>
   </link>
