Commit message: update: import stl file in MKS unit system
I wrote component.urdf to tune the offset of each STL file. After
getting the offsets and rotation, I replaced the simple geometry of
femur 1 and tibia 1 by stl files.

File: spyndra_description/urdf/spyndra.urdf.xacro (robot description, xacro)
@@ -3,4 +3,5 @@
   <!-- constants -->
   <xacro:property name="pi" value="3.1415926535897931"/>
+  <!-- stl offset -->
   <!-- component length -->
   <xacro:property name="lc1" value="0.068"/>
@@ -32,23 +33,18 @@
     <collision>
       <geometry>
-        <box size="${2*lc1} ${2*lc1} ${hc1}" />
-      </geometry>
-      <origin rpy="0 0 0" xyz="0 0 ${hc1/2}"/>
-    </collision>
-    <visual>
-      <geometry>
-        <box size="${2*lc1} ${2*lc1} ${hc1}" />
-      </geometry>
+        <mesh filename="package://spyndra_description/meshes/chassis.stl"     scale="0.001 0.001 0.001"/>
+      </geometry>
+      <origin xyz="-0.11 -0.068 0" rpy="0 0 0"/>
+    </collision>
+    <visual>
+      <geometry>
+        <mesh filename="package://spyndra_description/meshes/chassis.stl"     scale="0.001 0.001 0.001"/>
+      </geometry>
+      <origin xyz="-0.11 -0.068 0" rpy="0 0 0"/>
       <material name="black"/>
-      <origin rpy="0 0 0" xyz="0 0 ${hc1/2}"/>
     </visual>
     <inertial>
       <origin xyz="0 0 ${hc1}"  rpy="0 0 0"/>
       <mass value="${mc}"/>
-      <!-- Simple geometry -->
-      <!--inertia ixx="${mc/12*(4*lc1*lc1+hc1*hc1)}" ixy="0"
-        iyy="${mc/12*(4*lc1*lc1+hc1*hc1)}" iyz="0"
-        izz="${mc/6*4*lc1*lc1}" ixz="0"/-->
-      <!-- From CAD file -->
       <inertia ixx="0.00029636" ixy="0.00000019"
         iyy="0.00028197" iyz = "-0.00000269"
@@ -59,24 +55,19 @@
     <collision>
       <geometry>
-        <box size="${lf} ${wf} ${hf}"/>
-      </geometry>
-      <material name="red"/>
-      <origin xyz="${lf/2} 0 0" rpy="0 0 0"/>
-    </collision>
-    <visual>
-      <geometry>
-        <box size="${lf} ${wf} ${hf}"/>
-      </geometry>
-      <material name="red"/>
-      <origin xyz="${lf/2} 0 0" rpy="0 0 0"/>
+        <mesh filename="package://spyndra_description/meshes/femur.stl"     scale="0.001 0.001 0.001"/>
+      </geometry>
+      <material name="red"/>
+      <origin xyz="-0.00825 0.0455 -0.022" rpy="3.1415926 -1.57075 0    "/>
+    </collision>
+    <visual>
+      <geometry>
+        <mesh filename="package://spyndra_description/meshes/femur.stl"     scale="0.001 0.001 0.001"/>
+      </geometry>
+      <material name="red"/>
+      <origin xyz="-0.00825 0.0455 -0.022" rpy="3.1415926 -1.57075 0    "/>
     </visual>
     <inertial>
       <origin xyz="${lf/2} 0 0" rpy="0 0 0"/>
       <mass value="${mf}"/>
-      <!-- Simple geometry -->
-      <!--inertia ixx="${mf/12*(wf*wf+hf*hf)}" ixy="0"
-        iyy="${mf/3*lf*lf+mf/12*wf*wf}" iyz="0"
-        izz="${mf/3*lf*lf+mf/12*hf*hf}" ixz="0"/-->
-      <!-- From CAD file -->
       <inertia ixx="${0.00025261+mf*(fy*fy+fz*fz)}"
         ixy="${        0.0-mf*fx*fy}"
@@ -90,24 +81,19 @@
     <collision>
       <geometry>
-        <cylinder length="${lt}" radius="${rt}"/>
-      </geometry>
-      <material name="white"/>
-      <origin rpy="0 ${pi/2} 0" xyz="${lt/2} 0 0"/>
-    </collision>
-    <visual>
-      <geometry>
-        <cylinder length="${lt}" radius="${rt}"/>
-      </geometry>
-      <material name="white"/>
-      <origin rpy="0 ${pi/2} 0" xyz="${lt/2} 0 0"/>
+        <mesh filename="package://spyndra_description/meshes/tibia.stl"     scale="0.001 0.001 0.001"/>
+      </geometry>
+      <material name="white"/>
+      <origin xyz="0.1735 0.0215 -0.02" rpy="1.57075 0 -1.57075"/>
+    </collision>
+    <visual>
+      <geometry>
+        <mesh filename="package://spyndra_description/meshes/tibia.stl"     scale="0.001 0.001 0.001"/>
+      </geometry>
+      <material name="white"/>
+      <origin xyz="0.1735 0.0215 -0.02" rpy="1.57075 0 -1.57075"/>
     </visual>
     <inertial>
       <origin xyz="${lt/2} 0 0" rpy="0 0 0"/>
       <mass value="${mt}"/>
-      <!-- Simple geometry -->
-      <!--inertia ixx="${mt/2*rt*rt}" ixy="0"
-        iyy="${mt/3*lt*lt}" iyz="0"
-        izz="${mt/3*lt*lt}" ixz="0"/ -->
-      <!-- From CAD file -->
       <inertia ixx="${0.00021435+mt*(ty*ty+tz*tz)}"
         ixy="${-0.00000128-mt*tx*ty}"

Commit message: delete redundant xacro parameters and add imu information
1. Renamed several xacro parameteres
2. Add xyzOffset and rpyOffset to Imu plugin
3. Reduced simulation rate of test_api
4. Reduced proportional gain of the PID controllers

Following works include
1. Calibrate positions of COM of chassis, femur and tibia.
2. Calibrate position of the imu sensor

File: spyndra_description/urdf/spyndra.urdf.xacro (robot description, xacro)
@@ -3,17 +3,5 @@
   <!-- constants -->
   <xacro:property name="pi" value="3.1415926535897931"/>
-  <!-- stl offset -->
-  <!-- component length -->
-  <xacro:property name="lc1" value="0.061"/>
-  <xacro:property name="lc2" value="0.058"/>
-  <xacro:property name="hc1" value="0.09441"/>
-  <xacro:property name="hc2" value="0.01"/>
-  <xacro:property name="lf" value="0.127"/>
-  <xacro:property name="wf" value="0.0848"/>
-  <xacro:property name="hf" value="0.06"/>
-  <xacro:property name="lt" value="0.18858"/>
-  <xacro:property name="rt" value="0.017"/>
-  <xacro:property name="dt" value="0.21227"/>
-  <!-- link offset -->
+  <!-- link offset for each STL file -->
   <xacro:property name="off_cx" value="-0.11" />
   <xacro:property name="off_cy" value="-0.068" />
@@ -25,5 +13,5 @@
   <xacro:property name="off_ty" value="0.0215" />
   <xacro:property name="off_tz" value="-0.02" />
-  <!-- joint offset -->
+  <!-- joint position -->
   <xacro:property name="jt_cx" value="0.0585" />
   <xacro:property name="jt_cy" value="-0.003" />
@@ -36,11 +24,28 @@
   <xacro:property name="mf" value="0.20096365"/>
   <xacro:property name="mt" value="0.10764861"/>
-  <!-- inertia offsets -->
-  <xacro:property name="fx" value="-0.0006" />
-  <xacro:property name="fy" value="0.0" />
-  <xacro:property name="fz" value="-0.05762" />
-  <xacro:property name="tx" value="-0.06001" />
-  <xacro:property name="ty" value="0.0" />
-  <xacro:property name="tz" value="0.0102" />
+  <!-- TODO: center of mass -->
+  <xacro:property name="chassis_origin_z" value="0.09441"/>
+  <xacro:property name="femur_origin_x" value="0.0635"/>
+  <xacro:property name="tibia_origin_x" value="0.09429"/>
+  <xacro:property name="femur_origin_z" value="0.09441"/>
+  <!-- moment of inertia -->
+  <xacro:property name="chassis_ixx" value="0.0029636" />
+  <xacro:property name="chassis_ixy" value="0.00000019" />
+  <xacro:property name="chassis_iyy" value="0.00028197" />
+  <xacro:property name="chassis_iyz" value="-0.00000269" />
+  <xacro:property name="chassis_izz" value="0.00044786" />
+  <xacro:property name="chassis_ixz" value="-0.00000106" />
+  <xacro:property name="femur_ixx" value="0.00025261" />
+  <xacro:property name="femur_ixy" value="0.0" />
+  <xacro:property name="femur_iyy" value="0.00014944" />
+  <xacro:property name="femur_iyz" value="-0.00000002" />
+  <xacro:property name="femur_izz" value="0.00013756" />
+  <xacro:property name="femur_ixz" value="-0.00000601" />
+  <xacro:property name="tibia_ixx" value="0.00021435" />
+  <xacro:property name="tibia_ixy" value="-0.00000128" />
+  <xacro:property name="tibia_iyy" value="0.00019560" />
+  <xacro:property name="tibia_iyz" value="-0.00005856" />
+  <xacro:property name="tibia_izz" value="0.00004159" />
+  <xacro:property name="tibia_ixz" value="0.00000606" />
   <!-- Import all Gazebo-customization elements -->
   <xacro:include filename="$(find spyndra_description)/urdf/spyndra.gazebo" />
@@ -62,9 +67,9 @@
     </visual>
     <inertial>
-      <origin xyz="0 0 ${hc1}"  rpy="0 0 0"/>
+      <origin xyz="0 0 ${chassis_origin_z}"  rpy="0 0 0"/>
       <mass value="${mc}"/>
-      <inertia ixx="0.00029636" ixy="0.00000019"
-        iyy="0.00028197" iyz = "-0.00000269"
-        izz="0.00044786" ixz="-0.00000106" />
+      <inertia ixx="${chassis_ixx}" ixy="${chassis_ixy}"
+        iyy="${chassis_iyy}" iyz = "${chassis_iyz}"
+        izz="${chassis_izz}" ixz="${chassis_ixz}" />
     </inertial>
   </link>
@@ -85,12 +90,9 @@
     </visual>
     <inertial>
-      <origin xyz="${lf/2} 0 0" rpy="0 0 0"/>
+      <origin xyz="${femur_origin_x} 0 ${femur_origin_z}" rpy="0 0 0"/>
       <mass value="${mf}"/>
-      <inertia ixx="${0.00025261+mf*(fy*fy+fz*fz)}"
-        ixy="${        0.0-mf*fx*fy}"
-        iyy="${ 0.00014944+mf*(fx*fx+fz*fz)}"
-        iyz="${-0.00000002-mf*fy*fz}"
-        izz="${ 0.00013756+mf*(fx*fx+fy*fy)}"
-        ixz="${-0.00000601-mf*fx*fz}" />
+      <inertia ixx="${femur_ixx}" ixy="${femur_ixy}"
+        iyy="${femur_iyy}" iyz = "${femur_iyz}"
+        izz="${femur_izz}" ixz="${femur_ixz}" />
     </inertial>
   </link>
@@ -111,12 +113,9 @@
     </visual>
     <inertial>
-      <origin xyz="${lt/2} 0 0" rpy="0 0 0"/>
+      <origin xyz="${tibia_origin_x} 0 0" rpy="0 0 0"/>
       <mass value="${mt}"/>
-      <inertia ixx="${0.00021435+mt*(ty*ty+tz*tz)}"
-        ixy="${-0.00000128-mt*tx*ty}"
-        iyy="${ 0.00019560+mt*(tx*tx+tz*tz)}"
-        iyz="${-0.00005856-mt*ty*tz}"
-        izz="${ 0.00004159+mt*(tx*tx+ty*ty)}"
-        ixz="${ 0.00000606-mt*tx*tz}" />
+      <inertia ixx="${tibia_ixx}" ixy="${tibia_ixy}"
+        iyy="${tibia_iyy}" iyz = "${tibia_iyz}"
+        izz="${tibia_izz}" ixz="${tibia_ixz}" />
     </inertial>
   </link>
@@ -137,12 +136,9 @@
     </visual>
     <inertial>
-      <origin xyz="0 0 ${hc1}"  rpy="0 0 0"/>
+      <origin xyz="${femur_origin_x} 0 ${femur_origin_z}"  rpy="0 0 0"/>
       <mass value="${mc}"/>
-      <inertia ixx="${0.00025261+mf*(fy*fy+fz*fz)}"
-        ixy="${        0.0-mf*fx*fy}"
-        iyy="${ 0.00014944+mf*(fx*fx+fz*fz)}"
-        iyz="${-0.00000002-mf*fy*fz}"
-        izz="${ 0.00013756+mf*(fx*fx+fy*fy)}"
-        ixz="${-0.00000601-mf*fx*fz}" />
+      <inertia ixx="${femur_ixx}" ixy="${femur_ixy}"
+        iyy="${femur_iyy}" iyz = "${femur_iyz}"
+        izz="${femur_izz}" ixz="${femur_ixz}" />
     </inertial>
   </link>
@@ -163,12 +159,9 @@
     </visual>
     <inertial>
-      <origin xyz="${lt/2} 0 0" rpy="0 0 0"/>
+      <origin xyz="${tibia_origin_x} 0 0" rpy="0 0 0"/>
       <mass value="${mt}"/>
-      <inertia ixx="${0.00021435+mt*(ty*ty+tz*tz)}"
-        ixy="${-0.00000128-mt*tx*ty}"
-        iyy="${ 0.00019560+mt*(tx*tx+tz*tz)}"
-        iyz="${-0.00005856-mt*ty*tz}"
-        izz="${ 0.00004159+mt*(tx*tx+ty*ty)}"
-        ixz="${ 0.00000606-mt*tx*tz}" />
+      <inertia ixx="${tibia_ixx}" ixy="${tibia_ixy}"
+        iyy="${tibia_iyy}" iyz = "${tibia_iyz}"
+        izz="${tibia_izz}" ixz="${tibia_ixz}" />
     </inertial>
   </link>
@@ -189,97 +182,78 @@
     </visual>
     <inertial>
-      <origin xyz="0 0 ${hc1}"  rpy="0 0 0"/>
+      <origin xyz="${femur_origin_x} 0 ${femur_origin_z}"  rpy="0 0 0"/>
       <mass value="${mc}"/>
-      <inertia ixx="${0.00025261+mf*(fy*fy+fz*fz)}"
-        ixy="${        0.0-mf*fx*fy}"
-        iyy="${ 0.00014944+mf*(fx*fx+fz*fz)}"
-        iyz="${-0.00000002-mf*fy*fz}"
-        izz="${ 0.00013756+mf*(fx*fx+fy*fy)}"
-        ixz="${-0.00000601-mf*fx*fz}" />
-    </inertial>
-    <inertial>
-      <origin xyz="${lt/2} 0 0" rpy="0 0 0"/>
+      <inertia ixx="${femur_ixx}" ixy="${femur_ixy}"
+        iyy="${femur_iyy}" iyz = "${femur_iyz}"
+        izz="${femur_izz}" ixz="${femur_ixz}" />
+    </inertial>
+  </link>
+  <link name="tibia_3">
+    <collision>
+      <geometry>
+        <mesh filename="package://spyndra_description/meshes/tibia.stl" scale="0.001 0.001 0.001"/>
+      </geometry>
+      <material name="white"/>
+      <origin xyz="${off_tx} ${off_ty} ${off_tz}" rpy="${pi/2} 0 ${-pi/2}"/>
+    </collision>
+    <visual>
+      <geometry>
+        <mesh filename="package://spyndra_description/meshes/tibia.stl" scale="0.001 0.001 0.001"/>
+      </geometry>
+      <material name="white"/>
+      <origin xyz="${off_tx} ${off_ty} ${off_tz}" rpy="${pi/2} 0 ${-pi/2}"/>
+    </visual>
+    <inertial>
+      <origin xyz="${tibia_origin_x} 0 0" rpy="0 0 0"/>
       <mass value="${mt}"/>
-      <inertia ixx="${mt/2*rt*rt}" ixy="0"
-        iyy="${mt/3*lt*lt}" iyz="0"
-        izz="${mt/3*lt*lt}" ixz="0"/>
-    </inertial>
-  </link>
-  <link name="tibia_3">
-    <collision>
-      <geometry>
-        <mesh filename="package://spyndra_description/meshes/tibia.stl" scale="0.001 0.001 0.001"/>
-      </geometry>
-      <material name="white"/>
-      <origin xyz="${off_tx} ${off_ty} ${off_tz}" rpy="${pi/2} 0 ${-pi/2}"/>
-    </collision>
-    <visual>
-      <geometry>
-        <mesh filename="package://spyndra_description/meshes/tibia.stl" scale="0.001 0.001 0.001"/>
-      </geometry>
-      <material name="white"/>
-      <origin xyz="${off_tx} ${off_ty} ${off_tz}" rpy="${pi/2} 0 ${-pi/2}"/>
-    </visual>
-    <inertial>
-      <origin xyz="${lt/2} 0 0" rpy="0 0 0"/>
+      <inertia ixx="${tibia_ixx}" ixy="${tibia_ixy}"
+        iyy="${tibia_iyy}" iyz = "${tibia_iyz}"
+        izz="${tibia_izz}" ixz="${tibia_ixz}" />
+    </inertial>
+  </link>
+  <link name="femur_4">
+    <collision>
+      <geometry>
+        <mesh filename="package://spyndra_description/meshes/femur.stl" scale="0.001 0.001 0.001"/>
+      </geometry>
+      <material name="red"/>
+      <origin xyz="${off_fx} ${off_fy} ${off_fz}" rpy="${pi} ${-pi/2} 0"/>
+    </collision>
+    <visual>
+      <geometry>
+        <mesh filename="package://spyndra_description/meshes/femur.stl" scale="0.001 0.001 0.001"/>
+      </geometry>
+      <material name="red"/>
+      <origin xyz="${off_fx} ${off_fy} ${off_fz}" rpy="${pi} ${-pi/2} 0"/>
+    </visual>
+    <inertial>
+      <origin xyz="${femur_origin_x} 0 ${femur_origin_z}"  rpy="0 0 0"/>
+      <mass value="${mc}"/>
+      <inertia ixx="${femur_ixx}" ixy="${femur_ixy}"
+        iyy="${femur_iyy}" iyz = "${femur_iyz}"
+        izz="${femur_izz}" ixz="${femur_ixz}" />
+    </inertial>
+  </link>
+  <link name="tibia_4">
+    <collision>
+      <geometry>
+        <mesh filename="package://spyndra_description/meshes/tibia.stl" scale="0.001 0.001 0.001"/>
+      </geometry>
+      <material name="white"/>
+      <origin xyz="${off_tx} ${off_ty} ${off_tz}" rpy="${pi/2} 0 ${-pi/2}"/>
+    </collision>
+    <visual>
+      <geometry>
+        <mesh filename="package://spyndra_description/meshes/tibia.stl" scale="0.001 0.001 0.001"/>
+      </geometry>
+      <material name="white"/>
+      <origin xyz="${off_tx} ${off_ty} ${off_tz}" rpy="${pi/2} 0 ${-pi/2}"/>
+    </visual>
+    <inertial>
+      <origin xyz="${tibia_origin_x} 0 0" rpy="0 0 0"/>
       <mass value="${mt}"/>
-      <inertia ixx="${0.00021435+mt*(ty*ty+tz*tz)}"
-        ixy="${-0.00000128-mt*tx*ty}"
-        iyy="${ 0.00019560+mt*(tx*tx+tz*tz)}"
-        iyz="${-0.00005856-mt*ty*tz}"
-        izz="${ 0.00004159+mt*(tx*tx+ty*ty)}"
-        ixz="${ 0.00000606-mt*tx*tz}" />
-    </inertial>
-  </link>
-  <link name="femur_4">
-    <collision>
-      <geometry>
-        <mesh filename="package://spyndra_description/meshes/femur.stl" scale="0.001 0.001 0.001"/>
-      </geometry>
-      <material name="red"/>
-      <origin xyz="${off_fx} ${off_fy} ${off_fz}" rpy="${pi} ${-pi/2} 0"/>
-    </collision>
-    <visual>
-      <geometry>
-        <mesh filename="package://spyndra_description/meshes/femur.stl" scale="0.001 0.001 0.001"/>
-      </geometry>
-      <material name="red"/>
-      <origin xyz="${off_fx} ${off_fy} ${off_fz}" rpy="${pi} ${-pi/2} 0"/>
-    </visual>
-    <inertial>
-      <origin xyz="0 0 ${hc1}"  rpy="0 0 0"/>
-      <mass value="${mc}"/>
-      <inertia ixx="${0.00025261+mf*(fy*fy+fz*fz)}"
-        ixy="${        0.0-mf*fx*fy}"
-        iyy="${ 0.00014944+mf*(fx*fx+fz*fz)}"
-        iyz="${-0.00000002-mf*fy*fz}"
-        izz="${ 0.00013756+mf*(fx*fx+fy*fy)}"
-        ixz="${-0.00000601-mf*fx*fz}" />
-    </inertial>
-  </link>
-  <link name="tibia_4">
-    <collision>
-      <geometry>
-        <mesh filename="package://spyndra_description/meshes/tibia.stl" scale="0.001 0.001 0.001"/>
-      </geometry>
-      <material name="white"/>
-      <origin xyz="${off_tx} ${off_ty} ${off_tz}" rpy="${pi/2} 0 ${-pi/2}"/>
-    </collision>
-    <visual>
-      <geometry>
-        <mesh filename="package://spyndra_description/meshes/tibia.stl" scale="0.001 0.001 0.001"/>
-      </geometry>
-      <material name="white"/>
-      <origin xyz="${off_tx} ${off_ty} ${off_tz}" rpy="${pi/2} 0 ${-pi/2}"/>
-    </visual>
-    <inertial>
-      <origin xyz="${lt/2} 0 0" rpy="0 0 0"/>
-      <mass value="${mt}"/>
-      <inertia ixx="${0.00021435+mt*(ty*ty+tz*tz)}"
-        ixy="${-0.00000128-mt*tx*ty}"
-        iyy="${ 0.00019560+mt*(tx*tx+tz*tz)}"
-        iyz="${-0.00005856-mt*ty*tz}"
-        izz="${ 0.00004159+mt*(tx*tx+ty*ty)}"
-        ixz="${ 0.00000606-mt*tx*tz}" />
+      <inertia ixx="${tibia_ixx}" ixy="${tibia_ixy}"
+        iyy="${tibia_iyy}" iyz = "${tibia_iyz}"
+        izz="${tibia_izz}" ixz="${tibia_ixz}" />
     </inertial>
   </link>
